File: phyduino_pico2_usbpd.kicad_sch (KiCad schematic)
At the start: 72 parts, among them J6 GT-USB-7047A, J9 GT-USB-7047A, Q1 SP30P25NQ, Q2 SP30P25NQ, U10 AP63205WU-7, U108 TPS2121RUXR, U109 TPS2121RUXR, U6 AP33772SDKZ-13-FA02, U8 AP63203WU-7, U9 TPUSBLC6-2P6

Commit message: nigthly commit
Other:
- company: (none) -> University of Toronto, Dept. of Physics
- title: (none) -> Phyduino Pico 2
Changed lines of the file:
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@@
 	(generator_version "10.0")
 	(paper "B")
+	(title_block
+		(title "Phyduino Pico 2")
+		(date "2026-05-04")
+		(rev "A")
+		(company "University of Toronto, Dept. of Physics")
+	)
 	(text "I_{LIMIT} = 2.6A"
 		(exclude_from_sim no)

Commit message: Made schematic changes : merged usb_pd sheet with wifi sheet. made system regulators adjustable.
Parts:
- removed C131, C132: 0.1µF, Capacitor_SMD [KL]:C_0402_1005Metric, symbol Device:C_Small
- removed C16, C24, C33, C35: 0.1μF, Capacitor_SMD [KL]:C_0805_2012Metric_Pad1.18x1.45mm_HandSolder, symbol Component - Device [KL]:C_Small
- removed C17, C18, C25, C27, C36: 22µF, Capacitor_SMD [KL]:C_0805_2012Metric_Pad1.18x1.45mm_HandSolder, symbol Component - Device [KL]:C_Small
- removed C19, C23, C29, C32: 10μF, Capacitor_SMD [KL]:C_0805_2012Metric_Pad1.18x1.45mm_HandSolder, symbol Component - Device [KL]:C_Small
- removed C28, C9: 0.1µF, Capacitor_SMD [KL]:C_1206_3216Metric_Pad1.33x1.80mm_HandSolder, symbol Component - Device [KL]:C_Small
- removed C30: 1µF, Capacitor_SMD [KL]:C_0402_1005Metric, symbol Component - Device [KL]:C_Small
- removed C31, C6: 0.1µF, Capacitor_SMD [KL]:C_0402_1005Metric, symbol Component - Device [KL]:C_Small
- removed J6, J9: GT-USB-7047A, Connector - PC SMT [UL]:GCT-USBC-GCT_USB4110, symbol KL - Connector:USB_C_Receptacle_USB2.0_16P
- removed L1: 3.3µH, Component - Inductor SMT [UL]:L_Bourns_SRP4021HMCT, symbol Inductor - Bourns:L_Bourns_SRP4021HMCT-3R3M
- removed L2: 4.7µH, Component - Inductor SMT [UL]:L_Bourns_SRP4021HMCT, symbol Inductor - Bourns:L_Bourns_SRP4021HMCT-4R7M
- removed Q1, Q2: SP30P25NQ, Package_DFN_QFN [KL]:Diodes_UDFN2020-6_Type-F, symbol UL - Transistors - MOSFET:PMPB27EP
- removed R10: 5mΩ, Resistor_SMD [KL]:R_0603_1608Metric, symbol Component - Device [KL]:R_Small
- removed R11, R12, R7, R8: 5.1kΩ, Resistor_SMD [KL]:R_0402_1005Metric, symbol Component - Device [KL]:R_Small
- removed R134: 42.2kΩ, Resistor_SMD [KL]:R_0402_1005Metric, symbol Device:R_Small
- removed R135, R138: 21kΩ, Resistor_SMD [KL]:R_0402_1005Metric, symbol Device:R_Small
- removed R136, R137: 5.1kΩ, Resistor_SMD [KL]:R_0402_1005Metric, symbol Device:R_Small
- removed R139, R141: 154kΩ, Resistor_SMD [KL]:R_0402_1005Metric, symbol Device:R_Small
- removed R140, R143, R144: 39.2kΩ, Resistor_SMD [KL]:R_0402_1005Metric, symbol Device:R_Small
- removed R142, R145: 10kΩ, Resistor_SMD [KL]:R_0402_1005Metric, symbol Device:R_Small
- removed R37, R47, R48: 5.1kΩ, Resistor_SMD [KL]:R_0402_1005Metric, symbol phyduino_pico:R_Small
- removed R40, R41: 100Ω, Resistor_SMD [KL]:R_0402_1005Metric, symbol phyduino_pico:R_Small
- removed R51: 47kΩ, Resistor_SMD [KL]:R_0805_2012Metric_Pad1.20x1.40mm_HandSolder, symbol phyduino_pico:R_Small
- removed R52: 16.5kΩ, Resistor_SMD [KL]:R_0805_2012Metric_Pad1.20x1.40mm_HandSolder, symbol phyduino_pico:R_Small
- removed R53: 111kΩ, Resistor_SMD [KL]:R_0805_2012Metric_Pad1.20x1.40mm_HandSolder, symbol phyduino_pico:R_Small
- removed R54: 18.7kΩ, Resistor_SMD [KL]:R_0805_2012Metric_Pad1.20x1.40mm_HandSolder, symbol phyduino_pico:R_Small
- removed R6, R9: 220kΩ, Resistor_SMD [KL]:R_0805_2012Metric_Pad1.20x1.40mm_HandSolder, symbol Component - Device [KL]:R_Small
- removed TH1: 10kΩ@25°C, Resistor_SMD [KL]:R_0402_1005Metric, symbol Component - Device [KL]:Thermistor_NTC
- removed TP10, TP11, TP13, TP18, TP2, TP22, TP4, TP5, TP6, TP7: TestPoint_Small, Component - Test point SMT [UL]:TestPoint_SameSky_CPG-47-TH-B, symbol Connector [KL]:TestPoint_Small
- removed U10: AP63205WU-7, Package_TO_SOT_SMD [KL]:TSOT-23-6_HandSoldering, symbol Power - Switching Regulator [KL]:AP63205WU
- removed U108, U109: TPS2121RUXR, Package - QFN [UL]:VQFN-HR-12, symbol PMIC - TI:TPS2121RUX
- removed U6: AP33772SDKZ-13-FA02, Package_DFN_QFN [KL]:QFN-24-1EP_4x4mm_P0.5mm_EP2.75x2.75mm, symbol Interface - USB:AP33772S
- removed U8: AP63203WU-7, Package_TO_SOT_SMD [KL]:TSOT-23-6_HandSoldering, symbol Power - Switching Regulator [KL]:AP63203WU
- removed U9: TPUSBLC6-2P6, Package_TO_SOT_SMD [KL]:SOT-666, symbol Protection - Signal:USBLC6-2P6
- removed Z3: ESDA25P35-1U1M-ES, Diode_SMD [KL]:ST_QFN-2L_1.6x1.0mm, symbol phyduino_pico:D_Zener_Filled
Connections:
- no-connect marks 16 -> 0
Other:
- note removed: ">1.06V"
- note removed: "I_{LIMIT} = 2.6A"
- note removed: "I_{LIMIT} = 2.7A"
- note removed: "Over Voltage = 22V"
- note removed: "Over Voltage = 5.5V"
- note removed: "V_{EN}=4.3V"
- note removed: "V_{EN}=7.0V"
- note removed: "V_{OVER} = 5.5V"
- note removed: "V_{USB_COMM} = +5.0V"
- note removed: "V_{USB_PD_OUT} = +5.0V to 20V"
