File: phyduino_pico2.kicad_pcb (KiCad board)
At the start: 4 copper layers, 68.6 x 53.3 mm, 166 parts, among them J1 1.0-3PWT, J2 PM2.54-1*8, J3 PM2.54-1*10, J4 PM2.54-1*6, J5 PM2.54-1*8, J6 GT-USB-7047A, J7 HC-FPC-0.5-22P-CSH20, J9 GT-USB-7047A, Q1 SP30P25NQ, Q2 SP30P25NQ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

Commit message: Updated board documentation.
Other:
- board text added: "LAYER 1"
- board text added: "LAYER 2"
- board text added: "LAYER 3"
- board text added: "LAYER 4"
