File: phyduino_pico2.kicad_pcb (KiCad board)
At the start: 4 copper layers, 68.6 x 53.3 mm, 179 parts, among them J1 1.0-3PWT, J2 PPPC081LFBN-RC, J3 PPPC101LFBN-RC, J4 PPPC061LFBN-RC, J5 PPPC081LFBN-RC, J6 GT-USB-7047A, J7 HC-FPC-0.5-22P-CSH20, J8 54-00127, J9 SM04B-SRSS-TB, SW1 1977067-1, U1 RP2350B, U10 AP63200WU, U108 TPS2121RUXR, U11 ESP32-C6-MINI-1-H4, U13 TPS259470ARPWR, U14 FXL6408UMX, U15 TPS3424C11EF2ADRLR, U2 AT25QF128A-SHB-T, U3 IS66WVR8M8FBLL-104NLI, U5 ADS7038QRTERQ1, U6 TPS259470ARPWR, U7 24AA64FT-I/MNY, U8 AP63200WU, U9 TPUSBLC6-2P6, Y1 ABM8G-12.000MHZ-18-D2Y-T

Commit message: Updated part numbers and distributor part nummbers after BoM review.
Parts:
- C14, C15: value 12pF -> 27pF
- C17, C18, C25, C36: footprint Capacitor_SMD:C_0805_2012Metric_Pad1.18x1.45mm_HandSolder -> Capacitor_SMD:C_1206_3216Metric_Pad1.33x1.80mm_HandSolder
- C9: footprint Capacitor_SMD:C_1206_3216Metric_Pad1.33x1.80mm_HandSolder -> Capacitor_SMD:C_1210_3225Metric
- D2: footprint Diode_SMD:D_TUMD2 -> Diode_SMD:D_SOD-323
- FB1: value ~ -> 1kΩ@100MHz
- FB100: value MLB1005F-221T -> MPZ1005S221HT000
- J1: value 1.0-3PWT -> SM03B-SRSS-TB
- J6: value GT-USB-7047A -> USB4110-GF-A
- J7: value HC-FPC-0.5-22P-CSH20 -> F32Q-1A7H1-11022
- R58: value 157kΩ -> 158kΩ
- U10, U8: value AP63200WU -> AP63301WU-7
- U3: value IS66WVR8M8FBLL-104NLI -> IS66WVS8M8FBLL-104NLI
- U5: value ADS7038QRTERQ1 -> ADS7038IRTER
- U7: value 24AA64FT-I/MNY -> AT24C64D-MAHM-T
- U9: value TPUSBLC6-2P6 -> USBLC6-2P6
- moved C17 0.25 mm to (55.7, 61.9)
- moved C18 0.25 mm to (55.7, 67.2)
- moved C25 0.25 mm to (67.0, 67.2)
- moved C36 0.25 mm to (67.0, 61.9)
- moved C9 0.25 mm to (32.7, 32.2)
Other:
- board text removed: "PROTOTYPE"
