File: phyduino2_power_regs.kicad_sch (KiCad schematic)
At the start: 58 parts, among them U10 AP63200WU, U108 TPS2121RUXR, U12 TPS259470ARPWR, U13 TPS259470ARPWR, U6 TPS259470ARPWR, U8 AP63200WU

Commit message: Development update : Initial design review changes and PCB routing.
Parts:
- C132, C137: value 0.033µF -> 0.1µF
- C136, C139: DIGIKEY PN 490-14514-1-ND -> (none); DIGKEY MANUFACTURER Murata Electronics -> (none); LCSC MANUFACTURER CCTC -> (none); LCSC PN C5142567 -> (none); PN TCC0402X7R104M500AT -> (none)
- C138, C140: DIGIKEY PN 490-14514-1-ND -> (none); DIGKEY MANUFACTURER Murata Electronics -> (none); LCSC MANUFACTURER CCTC -> (none); LCSC PN C5142567 -> (none); PN TCC0402X7R104M500AT -> (none); Variant ADV_SMT -> (none)
- R135, R138: value 21kΩ -> 42.2kΩ; DIGIKEY PN 311-21.0KLRCT-ND -> (none); DIGKEY MANUFACTURER YAGEO -> (none); LCSC MANUFACTURER FOJAN -> (none); LCSC PN C2998083 -> (none); PN FRC0402F2102TS -> (none)
- R136, R137: value 5.1kΩ -> 10kΩ; DIGIKEY PN 13-RC0402FR-7W5K1LCT-ND -> (none); DIGKEY MANUFACTURER YAGEO -> (none); LCSC MANUFACTURER CHANGLONG -> (none); LCSC PN CHANGLONG -> (none); PN CHANGLONG -> (none)
- R139, R146, R150, R151: DIGIKEY PN 13-RC0402FR-7W5K1LCT-ND -> (none); DIGKEY MANUFACTURER YAGEO -> (none); KiLib_Generator SMD_2terminal_chip_molded -> (none); LCSC MANUFACTURER CHANGLONG -> (none); LCSC PN CHANGLONG -> (none); PN CHANGLONG -> (none)
- R143, R147, R148, R149, R154, R155, R161: DIGIKEY PN 13-RC0402FR-7W5K1LCT-ND -> (none); DIGKEY MANUFACTURER YAGEO -> (none); LCSC MANUFACTURER CHANGLONG -> (none); LCSC PN CHANGLONG -> (none); PN CHANGLONG -> (none)
- R56, R57, R58, R59: DIGIKEY PN 311-47.0KCRCT-ND -> (none); DIGKEY MANUFACTURER YAGEO -> (none); LCSC MANUFACTURER UNI-ROYAL -> (none); LCSC PN C17713 -> (none); PN 0805W8F4702T5E -> (none); Variant STUDENT -> ADV_SMT
