File: phyduino2_power_regs.kicad_sch (KiCad schematic)
At the start: 58 parts, among them U10 AP63200WU, U108 TPS2121RUXR, U12 TPS259470ARPWR, U13 TPS259470ARPWR, U6 TPS259470ARPWR, U8 AP63200WU

Commit message: Development update : Schematic review changes (findings #6-#26).
- Pin map reworked onto 5 V-tolerant GPIOs; I2C1 shared by EEPROM,
  expander and J7 on GPIO38/39; UART1 shared by D0/D1 and ESP32 flashing.
- Power: U10 enable on GPIO33 (EN_5V) with VIN_MONITOR on GPIO43;
  VIN works like an Uno's (J2.8 on +V_EXTERNAL, U12 removed); C22 moved
  to +5.0V; C134 added on +V_EXTERNAL; C27 10 uF, C140 3.3 nF; notes
  corrected.
- A0-A5 protected with 1 kOhm arrays and 1 nF; R53 pull-down on WIFI_ENA;
  32 kHz labels removed; Y1 ABM8G with 12 pF load caps; I2C address
  notes corrected; Variants set on all parts.

Co-Authored-By: Claude Opus 5.5 <noreply@anthropic.com>
Parts:
- removed C137: 0.1µF, Capacitor_SMD:C_0402_1005Metric, symbol Device:C_Small
- removed C138: 1nF, Capacitor_SMD:C_0402_1005Metric, symbol Device:C_Small
- removed R147: 732kΩ, Resistor_SMD:R_0402_1005Metric, symbol Device:R_Small
- removed R148: 215kΩ, Resistor_SMD:R_0402_1005Metric, symbol Device:R_Small
- removed R151: 1.1kΩ, Resistor_SMD:R_0402_1005Metric, symbol Device:R_Small
- removed R159, R160: 10kΩ, Resistor_SMD:R_0402_1005Metric, symbol Device:R_Small
- removed R161: 53.6kΩ, Resistor_SMD:R_0402_1005Metric, symbol Device:R_Small
- removed U12: TPS259470ARPWR, Package - QFN [UL]:Texas_Instruments_VQFN-HR-10, symbol [UL] PMIC - eFuse:TPS259470ARPWR
- added C134: 1µF, Capacitor_SMD:C_0805_2012Metric_Pad1.18x1.45mm_HandSolder, symbol Device:C_Small
- added C141: 1nF, Capacitor_SMD:C_0402_1005Metric, symbol Device:C_Small
- added D2: 3.6V, Diode_SMD:D_TUMD2, symbol Device:D_Zener_Filled
- added R165: 100kΩ, Resistor_SMD:R_0402_1005Metric, symbol Device:R_Small
- added R166: 10kΩ, Resistor_SMD:R_0402_1005Metric, symbol Device:R_Small
- added TP10, TP14, TP18, TP19, TP23: TestPoint_Small, Component - Test point SMT [UL]:TestPoint_SameSky_CPG-47-TH-B, symbol Connector [KL]:TestPoint_Small
- C132: KiLib_Generator (none) -> SMD_2terminal_chip_molded; PN (none) -> TCC0402X7R104M500AT
- C139: PN (none) -> TCC0402X7R104M500AT
- C140: value 1nF -> 3300pF; Variant (none) -> ADV_SMT
- C22, C28, C8: KiLib_Generator (none) -> capacitor/SMD/elec_round
- C5, C7: KiLib_Generator (none) -> SMD_2terminal_chip_molded
- renumbered TP27 to TP17, TP22 to TP20
Connections:
- net +3.3V: now also TP14.1
- net +5.0V: now also C22.1, TP19.1
- net +EXTERNAL_POWER: now also C134.1, TP23.1
- net +VIN_REG: now also R165.2, TP18.1; no longer C22.1
- net +VUSB: now also TP10.1
- net GND: now also C134.2, C141.2, D2.2 (A), R166.1
- net SEL_5V: no longer U10.2 (EN)
- new net EN_5V: U10.2 (EN)
- new net VIN_MONITOR: C141.1, D2.1 (K), R165.1, R166.2
Other:
- note added: "Enables +5.0V DC/DC when +VIN_REG > 5.5V"
- note added: "NOTES: C_{dVdt} > 10nF, it is recommended to add a 100Ω resistor in series before capacitor"
- note removed: "- U10 will only enable when +VUSB is above +7.0V."
- note removed: "- U108 select between +VUSB and the output of U10. If both voltages are below +5.5V, U10's output will be selected."
- note removed: "- U8 will only enable when +VUSB is above +4.3V."
- note removed: "Enables +5.0V DC/DC when VIN2 > 6.0V"
- note removed: "NOTES:"
- note removed: "NOTES: C_{dVdt} > 10nF, it is recommended to 100Ω in series with capacitor"
- moved on the sheet: C139, C140, C23, C28, R149, R153, R154, R155, R156, R162, R163, TP17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
