File: phyduino2_power_regs.kicad_sch (KiCad schematic)
At the start: 59 parts, among them U10 AP63200WU, U108 TPS2121RUXR, U13 TPS259470ARPWR, U6 TPS259470ARPWR, U8 AP63200WU

Commit message: Resized schematic sheet to A from B. Add micropython logo to back silkscreen. Regenerated gerber files
Parts:
- added R151: 22kΩ, Resistor_SMD:R_0402_1005Metric, symbol Device:R_Small
- added R152: 33kΩ, Resistor_SMD:R_0402_1005Metric, symbol Device:R_Small
- C139: VOLTAGE (none) -> 16V
Connections:
- net +VUSB: now also R151.2
- net GND: now also R152.1
- new net VBUS_DETECT: R151.1, R152.2
Other:
- note added: "NOTES: - C_{dVdt} > 10nF, it is recommended to add a 100Ω resistor in series before capacitor"
- note removed: "NOTES: C_{dVdt} > 10nF, it is recommended to add a 100Ω resistor in series before capacitor"
- moved on the sheet: C131, C132, C134, C136, C139, C140, C141, C16, C17, C18, C19, C22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

Commit message: Updated part numbers and distributor part nummbers after BoM review.
Parts:
- C131: DIGIKEY PN 490-14514-1-ND -> (none); DIGIKEY_PN (none) -> 490-14514-1-ND; DIGKEY MANUFACTURER Murata Electronics -> (none); KiLib_Generator SMD_2terminal_chip_molded -> (none); LCSC MANUFACTURER CCTC -> (none); LCSC PN C5142567 -> (none); LCSC_PN (none) -> C85858; MOUSER_PN (none) -> 81-GCM155R71H104KE2J; PN TCC0402X7R104M500AT -> GCM155R71H104KE02J; Tolerance (none) -> ±10%
- C132: DIGIKEY_PN (none) -> 490-14514-1-ND; KiLib_Generator SMD_2terminal_chip_molded -> (none); LCSC_PN (none) -> C85858; MOUSER_PN (none) -> 81-GCM155R71H104KE2J; PN TCC0402X7R104M500AT -> GCM155R71H104KE02J; Tolerance ±5% -> ±10%; VOLTAGE 16V -> (none)
- C134: DIGIKEY_PN (none) -> 490-10675-1-ND; KiLib_Generator SMD_2terminal_chip_molded -> (none); LCSC_PN (none) -> C342759; MOUSER_PN (none) -> 81-GCM21BR71H105KA3L; PN (none) -> GCM21BR71H105KA03L; Tolerance ±5% -> ±10%; VOLTAGE 50V -> (none)
- C136, C141: DIGIKEY_PN (none) -> 490-3244-1-ND; KiLib_Generator SMD_2terminal_chip_molded -> (none); LCSC_PN (none) -> C76947; MOUSER_PN (none) -> 81-GRM1555C1H102JA1D; PN (none) -> GRM1555C1H102JA01D
- C139: DIGIKEY_PN (none) -> 490-14514-1-ND; KiLib_Generator SMD_2terminal_chip_molded -> (none); LCSC_PN (none) -> C85858; MOUSER_PN (none) -> 81-GCM155R71H104KE2J; PN TCC0402X7R104M500AT -> GCM155R71H104KE02J; Tolerance (none) -> ±10%; VOLTAGE 16V -> (none)
- C140: DIGIKEY_PN (none) -> 490-3248-1-ND; KiLib_Generator SMD_2terminal_chip_molded -> (none); LCSC_PN (none) -> C85963; MOUSER_PN (none) -> 81-GRM36X332K50; PN (none) -> GRM155R71H332KA01D
- C16, C24: DIGIKEY PN 1276-1003-1-ND -> (none); DIGIKEY_PN (none) -> 1276-1003-1-ND; DIGKEY MANUFACTURER Samsung Electro-Mechanics -> (none); KiLib_Generator SMD_2terminal_chip_molded -> (none); LCSC MANUFACTURER TORCH -> (none); LCSC PN C53084456 -> (none); LCSC_PN (none) -> C1711; MOUSER_PN (none) -> 187-CL21B104KBCNNNC; PN CC0805X7R50V104MN -> CL21B104KBCNNNC
- C17, C18, C36: footprint Capacitor_SMD:C_0805_2012Metric_Pad1.18x1.45mm_HandSolder -> Capacitor_SMD:C_1206_3216Metric_Pad1.33x1.80mm_HandSolder; DIGIKEY PN 1276-CL21A226MAYNNNECT-ND -> (none); DIGIKEY_PN (none) -> 445-6000-1-ND; DIGKEY MANUFACTURER Samsung Electro-Mechanics -> (none); KiLib_Generator SMD_2terminal_chip_molded -> (none); LCSC MANUFACTURER Chinocera -> (none); LCSC PN C22367832 -> (none); MOUSER_PN (none) -> 810-C3216X5R1E226M; PN HGC0805R5226M350NSLJ -> C3216X5R1E226M160AB; Tolerance (none) -> ±20%
- C19, C23: DIGIKEY PN 490-10748-1-ND -> (none); DIGIKEY_PN (none) -> 4713-GMC21X5R106K50NTCT-ND; DIGKEY MANUFACTURER Murata Electronics -> (none); KiLib_Generator SMD_2terminal_chip_molded -> (none); LCSC MANUFACTURER AIDE CAPACITOR -> (none); LCSC PN C49326680 -> (none); LCSC_PN (none) -> C440198; MOUSER_PN (none) -> 603-CC0805KKX59BB106; PN 0805X5R106K350NT -> GMC21X5R106K50NT
- C22, C28, C8: DIGIKEY_PN (none) -> 5011-VPXB0771E101MVTM-ND; KiLib_Generator capacitor/SMD/elec_round -> (none); MFR Ymin -> (none)
- C25: footprint Capacitor_SMD:C_0805_2012Metric_Pad1.18x1.45mm_HandSolder -> Capacitor_SMD:C_1206_3216Metric_Pad1.33x1.80mm_HandSolder; DIGIKEY PN 1276-CL21A226MAYNNNECT-ND -> (none); DIGIKEY_PN (none) -> 445-6000-1-ND; DIGKEY MANUFACTURER Samsung Electro-Mechanics -> (none); KiLib_Generator SMD_2terminal_chip_molded -> (none); LCSC MANUFACTURER Chinocera -> (none); LCSC PN C22367832 -> (none); MOUSER_PN (none) -> 810-C3216X5R1E226M; PN HGC0805R5226M350NSLJ -> C3216X5R1E226M160AB; Tolerance (none) -> ±20%; VOLTAGE (none) -> 25V
- C5, C7: DIGIKEY_PN (none) -> 1276-1025-1-ND; KiLib_Generator SMD_2terminal_chip_molded -> (none); LCSC_PN (none) -> C26409; MOUSER_PN (none) -> 187-CL05C101JB5NNNC; PN (none) -> CL05C101JB5NNNC
- D2: footprint Diode_SMD:D_TUMD2 -> Diode_SMD:D_SOD-323; DIGIKEY_PN (none) -> MM3Z3V6T1GOSCT-ND; LCSC_PN (none) -> C116949; MFR Rohm Semiconductor -> (none); MOUSER_PN (none) -> 863-MM3Z3V6T1G; PN TFZVTR3.6B -> MM3Z3V6T1G
- L1: DIGIKEY PN 118-SRP4021HMCT-6R8MCT-ND -> (none); DIGIKEY_PN (none) -> 118-SRP4021HMCT-6R8MCT-ND; DIGKEY MANUFACTURER Bourns Inc. -> (none); LCSC MANUFACTURER BOURNS -> (none); MOUSER_PN (none) -> 652-SRP4021HMCT-6R8M
- L2: DIGIKEY PN 118-SRP4021HMCT-100MCT-ND -> (none); DIGIKEY_PN (none) -> 118-SRP4021HMCT-100MCT-ND; DIGKEY MANUFACTURER Bourns Inc. -> (none); LCSC MANUFACTURER BOURNS -> (none); MOUSER_PN (none) -> 652-SRP4021HMCT-100M
- R134: DIGIKEY PN 311-42.2KLRCT-ND -> (none); DIGIKEY_PN (none) -> 311-42.2KLRCT-ND; DIGKEY MANUFACTURER YAGEO -> (none); KiLib_Generator SMD_2terminal_chip_molded -> (none); LCSC MANUFACTURER RALEC -> (none); LCSC PN C103034 -> (none); LCSC_PN (none) -> C276270; MOUSER_PN (none) -> 603-RC0402FR-0742K2L; PN RTT024222FTH -> RC0402FR-0742K2L
- R135, R138: DIGIKEY_PN (none) -> 311-42.2KLRCT-ND; KiLib_Generator SMD_2terminal_chip_molded -> (none); LCSC_PN (none) -> C276270; MOUSER_PN (none) -> 603-RC0402FR-0742K2L; PN (none) -> RC0402FR-0742K2L
- R136, R137: DIGIKEY_PN (none) -> 311-10.0KLRCT-ND; KiLib_Generator SMD_2terminal_chip_molded -> (none); LCSC_PN (none) -> C60490; MOUSER_PN (none) -> 603-RC0402FR-0710KL; PN (none) -> RC0402FR-0710KL
- R139: DIGIKEY_PN (none) -> 311-1.10KLRCT-ND; LCSC_PN (none) -> C2909306; MOUSER_PN (none) -> 603-RC0402FR-071K1L; PN (none) -> RC0402FR-071K1L
- R143, R149: DIGIKEY_PN (none) -> YAG3224CT-ND; KiLib_Generator SMD_2terminal_chip_molded -> (none); LCSC_PN (none) -> C5159692; MOUSER_PN (none) -> 603-RC0402FR-07732KL; PN (none) -> RC0402FR-07732KL
- R146: DIGIKEY_PN (none) -> YAG3055CT-ND; LCSC_PN (none) -> C11489; MOUSER_PN (none) -> 603-RC0402FR-07215KL; PN (none) -> RC0402FR-07215KL
- R150: DIGIKEY_PN (none) -> 311-53.6KLRCT-ND; LCSC_PN (none) -> C5153961; MOUSER_PN (none) -> 603-RC0402FR-0753K6L; PN (none) -> RC0402FR-0753K6L
- R151: DIGIKEY_PN (none) -> P22.0KLCT-ND; KiLib_Generator SMD_2terminal_chip_molded -> (none); LCSC_PN (none) -> C413100; MOUSER_PN (none) -> 603-RC0402FR-0722KL; PN (none) -> ERJ-2RKF2202X
- R152: DIGIKEY_PN (none) -> 311-33.0KLRCT-ND; KiLib_Generator SMD_2terminal_chip_molded -> (none); LCSC_PN (none) -> C25779; MOUSER_PN (none) -> 603-RC0402FR-0733KL; PN (none) -> RC0402FR-0733KL
- R153, R157, R158, R162, R163, R166: DIGIKEY PN 311-10.0KLRCT-ND -> (none); DIGIKEY_PN (none) -> 311-10.0KLRCT-ND; DIGKEY MANUFACTURER YAGEO -> (none); KiLib_Generator SMD_2terminal_chip_molded -> (none); LCSC MANUFACTURER FOJAN -> (none); LCSC PN C2906861 -> (none); LCSC_PN (none) -> C60490; MOUSER_PN (none) -> 603-RC0402FR-0710KL; PN FRC0402F1002TS -> RC0402FR-0710KL
- R154: DIGIKEY_PN (none) -> 311-53.6KLRCT-ND; KiLib_Generator SMD_2terminal_chip_molded -> (none); LCSC_PN (none) -> C5153961; MOUSER_PN (none) -> 603-RC0402FR-0753K6L; PN (none) -> RC0402FR-0753K6L
- R155: DIGIKEY_PN (none) -> YAG3055CT-ND; KiLib_Generator SMD_2terminal_chip_molded -> (none); LCSC_PN (none) -> C11489; MOUSER_PN (none) -> 603-RC0402FR-07215KL; PN (none) -> RC0402FR-07215KL
- R156: DIGIKEY PN 13-RC0402FR-7W5K1LCT-ND -> (none); DIGIKEY_PN (none) -> 311-1.10KLRCT-ND; DIGKEY MANUFACTURER YAGEO -> (none); KiLib_Generator SMD_2terminal_chip_molded -> (none); LCSC MANUFACTURER CHANGLONG -> (none); LCSC PN CHANGLONG -> (none); LCSC_PN (none) -> C2909306; MOUSER_PN (none) -> 603-RC0402FR-071K1L; PN CHANGLONG -> RC0402FR-071K1L
- R165: DIGIKEY PN 311-10.0KLRCT-ND -> (none); DIGIKEY_PN (none) -> 311-100KLRCT-ND; DIGKEY MANUFACTURER YAGEO -> (none); KiLib_Generator SMD_2terminal_chip_molded -> (none); LCSC MANUFACTURER FOJAN -> (none); LCSC PN C2906861 -> (none); LCSC_PN (none) -> C60491; MOUSER_PN (none) -> 603-RC0402FR-07100KL; PN FRC0402F1002TS -> RC0402FR-07100KL
- R56: DIGIKEY_PN (none) -> YAG3024CT-ND; KiLib_Generator SMD_2terminal_chip_molded -> (none); LCSC_PN (none) -> C26996; MOUSER_PN (none) -> 603-RC0402FR-07196KL; PN (none) -> RC0402FR-07196KL
- R57: DIGIKEY_PN (none) -> 311-62.0KLRCT-ND; KiLib_Generator SMD_2terminal_chip_molded -> (none); LCSC_PN (none) -> C2909375; MOUSER_PN (none) -> 603-RC0402FR-0762KL; PN (none) -> RC0402FR-0762KL
- R58: value 157kΩ -> 158kΩ; DIGIKEY_PN (none) -> YAG2990CT-ND; KiLib_Generator SMD_2terminal_chip_molded -> (none); LCSC_PN (none) -> C4014665; MOUSER_PN (none) -> 603-RC0402FR-07158KL; PN (none) -> RC0402FR-07158KL
- R59: DIGIKEY_PN (none) -> 311-30.0KLRCT-ND; KiLib_Generator SMD_2terminal_chip_molded -> (none); LCSC_PN (none) -> C138008; MOUSER_PN (none) -> 603-RC0402FR-0730KL; PN (none) -> RC0402FR-0730KL
- U10, U8: value AP63200WU -> AP63301WU-7; DIGIKEY_PN (none) -> 31-AP63301WU-7CT-ND; LCSC_PN (none) -> C2158003; MOUSER_PN (none) -> 621-AP63301WU-7; PN (none) -> ${VALUE}
- U108: DIGIKEY PN 296-53410-1-ND -> (none); DIGIKEY_PN (none) -> 296-53410-1-ND; DIGKEY MANUFACTURER Texas Instruments -> (none); LCSC MANUFACTURER Texas Instruments -> (none); LCSC PN C485916 -> (none); LCSC_PN (none) -> C485916; MOUSER_PN (none) -> 595-TPS2121RUXR
- U13, U6: DIGIKEY_PN (none) -> 296-TPS259470ARPWRCT-ND; MOUSER_PN (none) -> 595-TPS259470ARPWR; PN (none) -> ${VALUE}
