File: phyduino_pico2_mcu.kicad_sch (KiCad schematic)
At the start: 68 parts, among them J1 1.0-3PWT, SW1 1977067-1, SW2 MINI MSK12CO2, U1 RP2350B, U2 GD25LQ128EWIGR, U3 PCA9570GMH, U4 XC6190AN157R-G, U5 ADS7038QRTERQ1, U7 ZD24C64A-MAGMT, Y1 XC32M4-12.000-F10NNFT

Commit message: Built board without USB-PD variant. Not yet complete.
Parts:
- removed C22: 0.1µF, Capacitor_SMD [KL]:C_0402_1005Metric, symbol phyduino_pico:C_Small
- removed RN1: 3.3kΩ, Resistor_SMD [KL]:R_Array_Convex_4x0603, symbol Component - Resistor Network:CAT16-3301F4LF
- removed U2: GD25LQ128EWIGR, Package - DFN [UL]:DFN-8-1EP_5x6mm_P1.27mm_3.6x4.2mm, symbol Digital - Memory - Flash:AT25QF128A-MHB-T
- removed U3: PCA9570GMH, Package - QFN [UL]:XQFN-8_1.6x1.6mm_P0.5mm, symbol Digital - IO Expanders:PCA9750
- added C6: 0.1µF, Capacitor_SMD:C_0402_1005Metric, symbol Component - Device [KL]:C_Small
- added R53, R54, R60, R63: 1.1kΩ, Resistor_SMD:R_0402_1005Metric, symbol phyduino_pico:R_Small
- added R61, R62: 4.7kΩ, Resistor_SMD:R_0402_1005Metric, symbol phyduino_pico:R_Small
- added U2: GD25LE128EXHIGR, Package - SON [UL]:USON-8-2EP_3x3mm_P0.8mm_EP0.8x.02mm, symbol [UL] Digital - Memory - Flash:GD25LE128EXHIGR
- added U3: IS66WVR8M8FBLL-104NLI, Package_SO:SOIC-8_3.9x4.9mm_P1.27mm, symbol [UL] Digital - Memory - RAM:IS66WVR8M8FBLL-104NLI
- C1, C110, C111, C117, C119, C120, C125, C126, C129, C130, C133, C135, C14, C15, C2, C20, C21, C26, C3, C34, C4, C57: footprint Capacitor_SMD [KL]:C_0402_1005Metric -> Capacitor_SMD:C_0402_1005Metric
- C10, C11, C12: footprint Capacitor_SMD [KL]:C_0402_1005Metric -> Capacitor_SMD:C_0805_2012Metric_Pad1.18x1.45mm_HandSolder
- D1: footprint LED_SMD [KL]:LED_0603_1608Metric -> LED_SMD:LED_0805_2012Metric_Pad1.15x1.40mm_HandSolder
- D2, D5: value GREEN -> RED; footprint LED_SMD [KL]:LED_0805_2012Metric_Pad1.15x1.40mm_HandSolder -> LED_SMD:LED_0805_2012Metric_Pad1.15x1.40mm_HandSolder; DIGIKEY PN 732-4986-1-ND -> 732-4971-1-ND; LCSC MANUFACTURER CHONGTIAN -> EVERLIGHT; LCSC PN C52676048 -> C2986048; PN CT-2012UGC-P8 -> 19-21/GHC-YR1S2/4T; Variant STUDENT -> ADV_SMT
- D3: value GREEN -> ORANGE; footprint LED_SMD [KL]:LED_0805_2012Metric_Pad1.15x1.40mm_HandSolder -> LED_SMD:LED_0805_2012Metric_Pad1.15x1.40mm_HandSolder; DIGIKEY PN 732-4986-1-ND -> 732-4971-1-ND; LCSC MANUFACTURER CHONGTIAN -> EVERLIGHT; LCSC PN C52676048 -> C2986048; PN CT-2012UGC-P8 -> 19-21/GHC-YR1S2/4T; Variant STUDENT -> ADV_SMT
- D4: footprint LED_SMD [KL]:LED_0805_2012Metric_Pad1.15x1.40mm_HandSolder -> LED_SMD:LED_0805_2012Metric_Pad1.15x1.40mm_HandSolder; DIGIKEY PN 732-4986-1-ND -> 732-4971-1-ND; LCSC MANUFACTURER CHONGTIAN -> EVERLIGHT; LCSC PN C52676048 -> C2986048; PN CT-2012UGC-P8 -> 19-21/GHC-YR1S2/4T; Variant STUDENT -> ADV_SMT
- FB1: footprint Inductor_SMD [KL]:L_0402_1005Metric -> Inductor_SMD:L_0805_2012Metric_Pad1.05x1.20mm_HandSolder
- FB100: footprint Inductor_SMD [KL]:L_0402_1005Metric -> Inductor_SMD:L_0402_1005Metric
- R1, R2: value 100Ω -> 100Ω; footprint Resistor_SMD [KL]:R_0402_1005Metric -> Resistor_SMD:R_0402_1005Metric
- R13, R3, R4, R46, R5: footprint Resistor_SMD [KL]:R_0402_1005Metric -> Resistor_SMD:R_0402_1005Metric
- R18, R20: value 10kΩ -> 10kΩ; footprint Resistor_SMD [KL]:R_0402_1005Metric -> Resistor_SMD:R_0402_1005Metric
- R42, R43: value 1.1kΩ -> 4.7kΩ; footprint Resistor_SMD [KL]:R_0402_1005Metric -> Resistor_SMD:R_0402_1005Metric
- R49: value 5.1kΩ -> 5.1kΩ; footprint Resistor_SMD [KL]:R_0402_1005Metric -> Resistor_SMD:R_0402_1005Metric
Connections:
- net +3.3V: now also C6.1, R61.1, R62.1, U2.8 (VCC), U3.8 (VDD)
- net BUILTIN_LED: now also U1.39 (GPIO31); no longer U1.47 (GPIO38)
- net D0: now also U1.42 (GPIO33); no longer U1.44 (GPIO35)
- net D1: now also U1.40 (GPIO32); no longer U1.43 (GPIO34)
- net D10: now also U1.56 (GPIO45); no longer U1.37 (GPIO29)
- net D11: now also U1.54 (GPIO43); no longer U1.39 (GPIO31)
- net D12: now also U1.55 (GPIO44); no longer U1.36 (GPIO28)
- net D13: now also U1.53 (GPIO42); no longer U1.38 (GPIO30)
- net D14: now also U1.57 (GPIO46); no longer U1.45 (GPIO36)
- net D15: now also U1.58 (GPIO47); no longer U1.46 (GPIO37)
- net D2: now also U1.43 (GPIO34); no longer U1.22 (GPIO22)
- net D3: now also U1.44 (GPIO35); no longer U1.23 (GPIO23)
- net D4: now also U1.45 (GPIO36); no longer U1.25 (GPIO24)
- net D5: now also U1.46 (GPIO37); no longer U1.26 (GPIO25)
- net D6: now also U1.47 (GPIO38); no longer U1.27 (GPIO26)
- net D7: now also U1.48 (GPIO39); no longer U1.28 (GPIO27)
- net D8: now also U1.49 (GPIO40); no longer U1.40 (GPIO32)
- net D9: now also U1.52 (GPIO41); no longer U1.42 (GPIO33)
- net FLASH_CLK: now also U2.6 (SCLK), U3.6 (CLK)
- net FLASH_SD0: now also U2.5 (SI), U3.5 (SI)
- net FLASH_SD1: now also U2.2 (SO), U3.2 (SO)
- net FLASH_SD2: now also U2.3 (WP#), U3.3 (SIO2)
- net FLASH_SD3: now also U2.7 (HOLD#), U3.7 (SIO3)
- net FLASH_~{CS}: now also U2.1 (CS#)
- net GND: now also C6.2, U2.4 (VSS), U3.4 (VSS)
- net PSW_STATUS: no longer U1.53 (GPIO42)
- net USBPD_FLIP: no longer U1.54 (GPIO43)
- net USBPD_GPIO: no longer U1.55 (GPIO44)
- net USBPD_INT: no longer U1.56 (GPIO45)
- net WIFI_DL_UART_RX: now also U1.37 (GPIO29); no longer U1.78 (GPIO1)
- net WIFI_DL_UART_TX: now also U1.36 (GPIO28); no longer U1.77 (GPIO0)
- net WIFI_ENA: now also U1.38 (GPIO30); no longer U1.4 (GPIO7)
- net WIFI_UART_CTS: now also U1.27 (GPIO26); no longer U1.8 (GPIO10)
- net WIFI_UART_RTS: now also U1.28 (GPIO27); no longer U1.9 (GPIO11)
- net WIFI_UART_RX: now also U1.26 (GPIO25); no longer U1.7 (GPIO9)
- net WIFI_UART_TX: now also U1.25 (GPIO24); no longer U1.6 (GPIO8)
- net WIFI_CONNECTED: now reaches D5.2 (A)
- net WIFI_CONNECTED: now also R63.2
- net USB_TX: now reaches D4.2 (A)
- net USB_TX: now also R60.2
- net USB_CONNECTED: now reaches D2.2 (A)
- net USB_CONNECTED: now also R53.2
- net TXD_COMM: now reaches U1.3 (GPIO6)
- net TXD_COMM: now also R60.1
- net USB_RX: now reaches D3.2 (A)
- net USB_RX: now also R54.2
- net HS_I2C0_SCL renamed I2C0_SDA
- net I2C0_SDA: now also TP1.1, U7.5 (SDA), R61.2
- net HS_I2C0_SDA renamed I2C0_SCL
- net I2C0_SCL: now also TP3.1, U7.6 (SCL), R62.2
- removed net I2C1_SCL: TP3.1, U1.58 (GPIO47), U7.6 (SCL)
- removed net I2C1_SDA: TP1.1, U1.57 (GPIO46), U7.5 (SDA)
- new net CONNECTED_COMM: R53.1, U1.6 (GPIO8)
- new net CONNECTED_WIFI: R63.1, U1.78 (GPIO1)
- new net HS_I2C1_SCL: U1.23 (GPIO23)
- new net HS_I2C1_SDA: U1.22 (GPIO22)
- new net PSRAM_CE#: U1.77 (GPIO0), U3.1 (CE#)
- new net RXD_COMM: R54.1, U1.4 (GPIO7)
Other:
- note added: "EEPROM"
- note removed: "I^{2}C Addr = 0x48"
- note removed: "Power Indicators & EEPROM"
- moved on the sheet: C1, C10, C11, C110, C111, C117, C119, C12, C120, C125, C126, C129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

Commit message: Development update : Changed the power input and tree, removed led for communication status.
Parts:
- removed D2, D5: RED, LED_SMD:LED_0805_2012Metric_Pad1.15x1.40mm_HandSolder, symbol Component - Device [KL]:LED_Filled
- removed D3: ORANGE, LED_SMD:LED_0805_2012Metric_Pad1.15x1.40mm_HandSolder, symbol Component - Device [KL]:LED_Filled
- removed D4: GREEN, LED_SMD:LED_0805_2012Metric_Pad1.15x1.40mm_HandSolder, symbol Component - Device [KL]:LED_Filled
- removed R53, R54, R60: 1.1kΩ, Resistor_SMD:R_0402_1005Metric, symbol phyduino_pico:R_Small
- added C29: 0.1µF, Capacitor_SMD:C_0402_1005Metric, symbol phyduino_pico:C_Small
- added R64: 10kΩ, Resistor_SMD:R_0402_1005Metric, symbol phyduino_pico:R_Small
- added U14: FXL6408UMX, Package - QFN [UL]:QFN40P260X180X55-16N, symbol [UL] Digital - IO Expanders:FXL6408UMX
- C10, C11, C12, D1, FB1: Variant ADV_SMT -> STUDENT
- R63: value 1.1kΩ -> 10kΩ
- SW2, U2: Variant (none) -> ADV_SMT
- TP1, TP12, TP15, TP19, TP20, TP21, TP23, TP24, TP25, TP26, TP3: Variant (none) -> IGNORE
- U3: Variant (none) -> STUDENT
Connections:
- net WIFI_CONNECTED is gone; now on net IO_EXP_~{INT}: R63.2
- net +3.3V: now also R63.1, C29.1, R64.1, U14.15 (VCC), U14.2 (VDDIO)
- net GND: now also C29.2, U14.16 (GND), U14.9 (ADDR)
- net I2C0_SCL: now also U14.13 (SCL)
- net I2C0_SDA: now also U14.14 (SDA)
- net PSW_STATUS: now also U14.3 (GPIO7)
- net CONNECTED_COMM: no longer names the net of U1.6 (GPIO8)
- net CONNECTED_WIFI: no longer names the net of U1.78 (GPIO1)
- net CONNECTED_WIFI: no longer R63.1
- net RXD_COMM renamed IO_EXP_~{RST}
- net IO_EXP_~{RST}: now also R64.2, U14.10 (~{RST})
- net TXD_COMM renamed IO_EXP_~{INT}
- net IO_EXP_~{INT}: now also U14.1 (~{INT})
- new net EXT_AUXOFF: U14.8 (GPIO2)
- new net EXT_~{FLT}: U14.11 (GPIO1)
- new net SHIELD_AUXOFF: U14.6 (GPIO4)
- new net SHIELD_~{FLT}: U14.7 (GPIO3)
- new net USB_AUXOFF: U14.4 (GPIO6)
- new net USB_~{FLT}: U14.5 (GPIO5)
- new net ~{EXT_PWR}: U14.12 (GPIO0)
Other:
- moved on the sheet: C1, C14, C15, C20, C21, C57, C6, J1, R1, R13, R18, R2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

Commit message: Development update : Initial design review changes and PCB routing.
Parts:
- removed R18: 10kΩ, Resistor_SMD:R_0402_1005Metric, symbol phyduino_pico:R_Small
- removed SW2: MINI MSK12CO2, Mechanical - Switch [UL]:Switch_Slide_ShouHan_MINI_MSK12CO2, symbol Mechanical - Switches:Slide_MINI_MSK12CO2
- removed TP25: TestPoint_Small, Component - Test point SMT [UL]:TestPoint_SameSky_CPG-47-TH-B, symbol Connector [KL]:TestPoint_Small
- removed U2: GD25LE128EXHIGR, Package - SON [UL]:USON-8-2EP_3x3mm_P0.8mm_EP0.8x.02mm, symbol [UL] Digital - Memory - Flash:GD25LE128EXHIGR
- removed U4: XC6190AN157R-G, Package - DFN [UL]:PHODET_VBPW34S, symbol UL - Digital logic:XC6190AN157R-G
- added C58: 4700pF, Capacitor_SMD:C_0402_1005Metric, symbol phyduino_pico:C_Small
- added C59: 1000pF, Capacitor_SMD:C_0402_1005Metric, symbol phyduino_pico:C_Small
- added R21, R22, R51, R52: 10kΩ, Resistor_SMD:R_0402_1005Metric, symbol phyduino_pico:R_Small
- added U15: TPS3424C11EF2ADRLR, Pacakge - SOT [UL]:SOT-5x3_DRL0008A_TEX, symbol [UL] PMIC - Supervisiors:TPS3434x11xxxADRLx
- added U2: AT25QF128A-SHB-T, Package_SO:SOIC-8_5.3x5.3mm_P1.27mm, symbol [UL] Digital - Memory - Flash:AT25QF128A-MHB-T
- C10, C11, C12: DIGIKEY PN 490-10017-1-ND -> (none); DIGKEY MANUFACTURER Murata Electronics -> (none); LCSC MANUFACTURER HRE -> (none); LCSC PN C49383783 -> (none); PN CSA0402X5R105M250GT -> (none)
- FB1: value MLB1005F-221T -> (none); DIGIKEY PN 445-6404-1-ND -> (none); DIGKEY MANUFACTURER TDK -> (none); LCSC MANUFACTURER MetalLions -> (none); LCSC PN C2844537 -> (none)
- R42, R43, R61, R62: value 4.7kΩ -> 5.1kΩ; DIGIKEY PN 13-RC0402FR-131K1LCT-ND -> (none); DIGKEY MANUFACTURER YAGEO -> (none); LCSC MANUFACTURER FOJAN -> (none); LCSC PN C2909306 -> (none); PN FRC0402F1101TS -> (none)
- R49: value 5.1kΩ -> 10kΩ
- R63, R64: DIGIKEY PN 13-RC0402FR-131K1LCT-ND -> (none); DIGKEY MANUFACTURER YAGEO -> (none); LCSC MANUFACTURER FOJAN -> (none); LCSC PN C2909306 -> (none); PN FRC0402F1101TS -> (none)
Connections:
- net BOOTMODE is gone; now on net FLASH_~{CS}: R49.1
- net SW_~{RESET} is gone; now on net EXT_~{RESET}: C57.1, SW1.2, TP26.1
- net +3.3V: now also R21.1, R22.1, R51.1, R52.2, U15.3 (VDD), U2.8 (VCC)
- net ADC_MISO: now also TP24.1, U1.55 (GPIO44); no longer TP20.1, U1.1 (GPIO4)
- net ADC_MOSI: now also U1.58 (GPIO47); no longer U1.80 (GPIO3)
- net ADC_SCK: now also TP20.1, U1.57 (GPIO46); no longer TP24.1, U1.79 (GPIO2)
- net ADC_nCS: now also U1.56 (GPIO45); no longer U1.2 (GPIO5)
- net BUILTIN_LED: now also U1.49 (GPIO40); no longer U1.39 (GPIO31)
- net D0: now also U1.80 (GPIO3); no longer U1.42 (GPIO33)
- net D1: now also U1.79 (GPIO2); no longer U1.40 (GPIO32)
- net D10: now also U1.21 (GPIO21); no longer U1.56 (GPIO45)
- net D11: now also U1.23 (GPIO23); no longer U1.54 (GPIO43)
- net D12: now also U1.20 (GPIO20); no longer U1.55 (GPIO44)
- net D13: now also U1.22 (GPIO22); no longer U1.53 (GPIO42)
- net D14: now also U1.25 (GPIO24); no longer U1.57 (GPIO46)
- net D15: now also U1.26 (GPIO25); no longer U1.58 (GPIO47)
- net D2: now also U1.1 (GPIO4); no longer U1.43 (GPIO34)
- net D3: now also U1.2 (GPIO5); no longer U1.44 (GPIO35)
- net D4: now also U1.3 (GPIO6); no longer U1.45 (GPIO36)
- net D5: now also U1.4 (GPIO7); no longer U1.46 (GPIO37)
- net D6: now also U1.6 (GPIO8); no longer U1.47 (GPIO38)
- net D7: now also U1.7 (GPIO9); no longer U1.48 (GPIO39)
- net D8: now also U1.8 (GPIO10); no longer U1.49 (GPIO40)
- net D9: now also U1.9 (GPIO11); no longer U1.52 (GPIO41)
- net EXT_AUXOFF: now also U14.5 (GPIO5); no longer U14.8 (GPIO2)
- net EXT_~{FLT}: now also U14.6 (GPIO4); no longer U14.11 (GPIO1)
- net EXT_~{RESET}: now also R22.2, U15.1 (PB)
- net FLASH_CLK: now also U2.6 (SCK)
- net FLASH_SD0: now also U2.5 (SI)
- net FLASH_SD1: now also U2.2 (SO)
- net FLASH_SD2: now also U2.3 (~{WP})
- net FLASH_SD3: now also U2.7 (~{HOLD})
- net FLASH_~{CS}: now also U2.1 (~{CS}); no longer R49.2
- net GND: now also C58.2, C59.2, U15.2 (GND), U2.4 (GND)
- net HS_I2C1_SCL: now also U1.48 (GPIO39); no longer U1.23 (GPIO23)
- net HS_I2C1_SDA: now also U1.47 (GPIO38); no longer U1.22 (GPIO22)
- net IO_EXP_~{INT}: now also U1.52 (GPIO41); no longer U1.3 (GPIO6)
- net IO_EXP_~{RST}: now also U1.45 (GPIO36); no longer U1.4 (GPIO7)
- net PSRAM_CE#: now also R51.2
- net PSW_STATUS: now also U14.8 (GPIO2); no longer U14.3 (GPIO7)
- net SHIELD_AUXOFF: now also U14.12 (GPIO0); no longer U14.6 (GPIO4)
- net SHIELD_~{FLT}: now also U14.11 (GPIO1); no longer U14.7 (GPIO3)
- net SYS_nRST: now also U15.7 (~{INT})
- net USB_AUXOFF: now also U14.3 (GPIO7); no longer U14.4 (GPIO6)
- net USB_~{FLT}: now also U14.4 (GPIO6); no longer U14.5 (GPIO5)
- net WIFI_DL_UART_RX: now also U1.28 (GPIO27); no longer U1.37 (GPIO29)
- net WIFI_DL_UART_TX: now also U1.27 (GPIO26); no longer U1.36 (GPIO28)
- net WIFI_ENA: now also U1.78 (GPIO1); no longer U1.38 (GPIO30)
- net WIFI_UART_CTS: now also U1.38 (GPIO30); no longer U1.27 (GPIO26)
- net WIFI_UART_RTS: now also U1.39 (GPIO31); no longer U1.28 (GPIO27)
- net WIFI_UART_RX: now also U1.37 (GPIO29); no longer U1.26 (GPIO25)
- net WIFI_UART_TX: now also U1.36 (GPIO28); no longer U1.25 (GPIO24)
- net ~{EXT_PWR}: now also U14.7 (GPIO3); no longer U14.12 (GPIO0)
- net I2C0_SCL renamed I2C1_SCL
- net I2C1_SCL: now also U1.54 (GPIO43); no longer U1.21 (GPIO21)
- net I2C0_SDA renamed I2C1_SDA
- net I2C1_SDA: now also U1.53 (GPIO42); no longer U1.20 (GPIO20)
- new net: R21.2, U15.8 (KILL)
- new net BOOT_LP_CAP: C58.1, U15.5 (LPT)
- new net MCU_BOOT_SEL: R49.2, R52.1, U15.6 (~{RESET})
- new net RESET_SP_CAP: C59.1, U15.4 (SPT)
- new net WIFI_BOOT1: U1.40 (GPIO32)
- no-connect marks 3 -> 2
Other:
- note added: "UART0 (F11)"
- note removed: "BOOT SWITCH - +3.3V Normal Boot mode - GND UF2 Boot mode"
- moved on the sheet: C1, C10, C11, C110, C111, C117, C119, C12, C120, C125, C126, C129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
