File: phyduino_pico2_mcu.kicad_sch (KiCad schematic)
At the start: 72 parts, among them J1 1.0-3PWT, SW1 1977067-1, U1 RP2350B, U14 FXL6408UMX, U15 TPS3424C11EF2ADRLR, U2 AT25QF128A-SHB-T, U3 IS66WVR8M8FBLL-104NLI, U5 ADS7038QRTERQ1, U7 ZD24C64A-MAGMT, Y1 XC32M4-12.000-F10NNFT

Commit message: Development update : Schematic review changes (findings #6-#26).
- Pin map reworked onto 5 V-tolerant GPIOs; I2C1 shared by EEPROM,
  expander and J7 on GPIO38/39; UART1 shared by D0/D1 and ESP32 flashing.
- Power: U10 enable on GPIO33 (EN_5V) with VIN_MONITOR on GPIO43;
  VIN works like an Uno's (J2.8 on +V_EXTERNAL, U12 removed); C22 moved
  to +5.0V; C134 added on +V_EXTERNAL; C27 10 uF, C140 3.3 nF; notes
  corrected.
- A0-A5 protected with 1 kOhm arrays and 1 nF; R53 pull-down on WIFI_ENA;
  32 kHz labels removed; Y1 ABM8G with 12 pF load caps; I2C address
  notes corrected; Variants set on all parts.

Co-Authored-By: Claude Opus 5.5 <noreply@anthropic.com>
Parts:
- added C30, C31, C32, C33, C35, C38: 1000pF, Capacitor_SMD:C_0402_1005Metric, symbol Component - Device [KL]:C_Small
- added RN1, RN2: 1.0kΩ, Component - Resistor Network:RESCAV50P200X100X55-8N, symbol Device:R_Pack04_Split
- added TP5: TestPoint_Small, Component - Test point SMT [UL]:TestPoint_SameSky_CPG-47-TH-B, symbol Connector [KL]:TestPoint_Small
- C14, C15: value 18pF -> 12pF; DIGIKEY PN 490-5858-1-ND -> (none); DIGKEY MANUFACTURER Murata Electronics -> (none); KiLib_Generator SMD_2terminal_chip_molded -> (none); LCSC MANUFACTURER YAGEO -> (none); LCSC PN C526984 -> (none); PN CC0402GRNPO8BN180 -> (none)
- C59: PN TCC0402X7R104M500AT -> (none)
- R13: value 1.1kΩ -> 620Ω
- U14, U15: Variant (none) -> ADV_SMT
- U2: KiLib_Generator (none) -> package/gullwing; Variant (none) -> ADV_SMT
- U3: KiLib_Generator (none) -> package/gullwing
- U7: value ZD24C64A-MAGMT -> 24AA64FT-I/MNY; DIGIKEY PN AT24C64D-MAHM-TCT-ND -> 24AA64FT-I/MNYCT-ND; FLASH_SIZE (none) -> 64kb; LCSC MANUFACTURER Zetta -> (none); LCSC PN C53284088 -> (none); Mem_Size 64Kb -> 64kb
- Y1: value XC32M4-12.000-F10NNFT -> ABM8G-12.000MHZ-18-D2Y-T; DIGIKEY PN 2151-H130B-12.000-18-3030-TRCT-ND -> 535-10261-1-ND; DIGKEY MANUFACTURER Raltron Electronics -> Abracon LLC; LCSC MANUFACTURER HCI -> (none); LCSC PN C2842186 -> (none)
- renumbered TP24 to TP12, TP21 to TP13, TP20 to TP15, TP23 to TP16, TP26 to TP22, TP3 to TP4, TP1 to TP6, TP12 to TP7, TP19 to TP8, TP15 to TP9
Connections:
- net HS_I2C1_SCL is gone; now on net I2C1_SCL: U1.48 (GPIO39)
- net HS_I2C1_SDA is gone; now on net I2C1_SDA: U1.47 (GPIO38)
- net A0: now also RN1.1 (R1.1); no longer U5.15 (AIN0/GPIO0)
- net A1: now also RN1.2 (R2.1); no longer U5.16 (AIN1/GPIO1)
- net A2: now also RN1.3 (R3.1); no longer U5.1 (AIN2/GPIO2)
- net A3: now also RN1.4 (R4.1); no longer U5.2 (AIN3/GPIO3)
- net A4: now also RN2.1 (R1.1); no longer U5.3 (AIN4/GPIO4)
- net A5: now also RN2.2 (R2.1); no longer U5.4 (AIN5/GPIO5)
- net D0: now also U1.2 (GPIO5); no longer U1.80 (GPIO3)
- net D1: now also U1.1 (GPIO4); no longer U1.79 (GPIO2)
- net D2: now also U1.79 (GPIO2); no longer U1.1 (GPIO4)
- net D3: now also U1.80 (GPIO3); no longer U1.2 (GPIO5)
- net GND: now also C30.2, C31.2, C32.2, C33.2, C35.2, C38.2
- net I2C1_SCL: no longer U1.54 (GPIO43)
- net I2C1_SDA: no longer U1.53 (GPIO42)
- net MCU_BOOT_SEL: now also TP5.1
- net EN_5V: now reaches U1.42 (GPIO33)
- net SHIELD_AUXOFF: no longer names the net of U14.12 (GPIO0)
- net SHIELD_~{FLT}: no longer names the net of U14.11 (GPIO1)
- new net AIN0: C30.1, RN1.8 (R1.2), U5.15 (AIN0/GPIO0)
- new net AIN1: C31.1, RN1.7 (R2.2), U5.16 (AIN1/GPIO1)
- new net AIN2: C32.1, RN1.6 (R3.2), U5.1 (AIN2/GPIO2)
- new net AIN3: C33.1, RN1.5 (R4.2), U5.2 (AIN3/GPIO3)
- new net AIN4: C35.1, RN2.8 (R1.2), U5.3 (AIN4/GPIO4)
- new net AIN5: C38.1, RN2.7 (R2.2), U5.4 (AIN5/GPIO5)
- new net VIN_MONITOR: U1.54 (GPIO43)
- no-connect marks 2 -> 12
Other:
- note added: "IO-EXPANDER"
- note added: "I^{2}C Addr = 0x43"
- note added: "I^{2}C Addr = 0x50"
- note removed: "I^{2}C Addr = 0x70"
- note removed: "UART0 (F11)"
- moved on the sheet: C1, C10, C11, C110, C111, C117, C119, C12, C120, C125, C126, C129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
