File: phyduino_pico2_mcu.kicad_sch (KiCad schematic)
At the start: 81 parts, among them J1 1.0-3PWT, SW1 1977067-1, U1 RP2350B, U14 FXL6408UMX, U15 TPS3424C11EF2ADRLR, U2 AT25QF128A-SHB-T, U3 IS66WVR8M8FBLL-104NLI, U5 ADS7038QRTERQ1, U7 24AA64FT-I/MNY, Y1 ABM8G-12.000MHZ-18-D2Y-T

Commit message: Resized schematic sheet to A from B. Add micropython logo to back silkscreen. Regenerated gerber files
Parts:
- removed C1, C6: 0.1µF, Capacitor_SMD:C_0402_1005Metric, symbol Component - Device [KL]:C_Small
- removed C10, C11, C12: 1µF, Capacitor_SMD:C_0805_2012Metric_Pad1.18x1.45mm_HandSolder, symbol Component - Device [KL]:C_Small
- removed C20, C21, C29, C57: 0.1µF, Capacitor_SMD:C_0402_1005Metric, symbol phyduino_pico:C_Small
- removed C30, C31, C32, C33, C35, C38: 1000pF, Capacitor_SMD:C_0402_1005Metric, symbol Component - Device [KL]:C_Small
- removed C58: 4700pF, Capacitor_SMD:C_0402_1005Metric, symbol phyduino_pico:C_Small
- removed C59: 1000pF, Capacitor_SMD:C_0402_1005Metric, symbol phyduino_pico:C_Small
- removed FB1: (no value), Inductor_SMD:L_0805_2012Metric_Pad1.05x1.20mm_HandSolder, symbol Component - Device [KL]:FerriteBead_Small
- removed R20, R21, R22, R49, R51, R52, R63, R64: 10kΩ, Resistor_SMD:R_0402_1005Metric, symbol phyduino_pico:R_Small
- removed R42, R43, R61, R62: 5.1kΩ, Resistor_SMD:R_0402_1005Metric, symbol phyduino_pico:R_Small
- removed RN1, RN2: 1.0kΩ, Component - Resistor Network:RESCAV50P200X100X55-8N, symbol Device:R_Pack04_Split
- removed SW1: 1977067-1, Mechanical - Switch [UL]:TE_1977067-1, symbol Mechanical - Switches:SW_Push_TE_1977067-1
- removed TP22, TP4, TP5, TP6: TestPoint_Small, Component - Test point SMT [UL]:TestPoint_SameSky_CPG-47-TH-B, symbol Connector [KL]:TestPoint_Small
- removed U14: FXL6408UMX, Package - QFN [UL]:QFN40P260X180X55-16N, symbol [UL] Digital - IO Expanders:FXL6408UMX
- removed U15: TPS3424C11EF2ADRLR, Pacakge - SOT [UL]:SOT-5x3_DRL0008A_TEX, symbol [UL] PMIC - Supervisiors:TPS3434x11xxxADRLx
- removed U2: AT25QF128A-SHB-T, Package_SO:SOIC-8_5.3x5.3mm_P1.27mm, symbol [UL] Digital - Memory - Flash:AT25QF128A-MHB-T
- removed U3: IS66WVR8M8FBLL-104NLI, Package_SO:SOIC-8_3.9x4.9mm_P1.27mm, symbol [UL] Digital - Memory - RAM:IS66WVR8M8FBLL-104NLI
- removed U5: ADS7038QRTERQ1, Package - QFN [UL]:QFN50P300X300X80-17N, symbol DAQ - ADC's:ADS7038-Q1
- removed U7: 24AA64FT-I/MNY, Package - DFN [UL]:DFN-8-1EP_3x2mm_P0.5mm_EP1.3x1.4mm, symbol Digital - Memory:24AA64FT-I/MNY
- added C127, C128, C137: 0.1µF, Capacitor_SMD:C_0402_1005Metric, symbol phyduino_pico:C_Small
- D1: footprint LED_SMD:LED_0805_2012Metric_Pad1.15x1.40mm_HandSolder -> LED_SMD:LED_0603_1608Metric; Variant STUDENT -> ADV_SMT
Connections:
- net +3.3V: now also C127.1, C128.1, C137.1
- net GND: now also C127.2, C128.2, C137.2
- net VBUS_DETECT: now reaches U1.43 (GPIO34)
- no-connect marks 12 -> 4
Other:
- added sheet Memory (phyduino_pico_memory.kicad_sch)
- added sheet Peripherals (phyduino_pico_peripherals.kicad_sch)
- note removed: "EEPROM"
- note removed: "External Analog-to-Digital Converter"
- note removed: "IO-EXPANDER"
- note removed: "I^{2}C Addr = 0x43"
- note removed: "I^{2}C Addr = 0x50"
- moved on the sheet: C110, C111, C117, C119, C120, C125, C126, C129, C130, C133, C135, C14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
