File: phyduino_pico2_mcu.kicad_sch (KiCad schematic)
At the start: 41 parts, among them J1 1.0-3PWT, U1 RP2350B, Y1 ABM8G-12.000MHZ-18-D2Y-T

Commit message: Updated part numbers and distributor part nummbers after BoM review.
Parts:
- C110, C111, C117, C119, C125, C126, C127, C128, C129, C130, C133, C135, C137, C26, C34: DIGIKEY PN 490-14514-1-ND -> (none); DIGIKEY_PN (none) -> 490-14514-1-ND; DIGKEY MANUFACTURER Murata Electronics -> (none); KiLib_Generator SMD_2terminal_chip_molded -> (none); LCSC MANUFACTURER CCTC -> (none); LCSC PN C5142567 -> (none); LCSC_PN (none) -> C85858; MOUSER_PN (none) -> 81-GCM155R71H104KE2J; PN TCC0402X7R104M500AT -> GCM155R71H104KE02J; Tolerance (none) -> ±10%
- C120, C2, C3, C4: DIGIKEY PN 490-GRM155C61E475ME15DCT-ND -> (none); DIGIKEY_PN (none) -> 445-13820-1-ND; DIGKEY MANUFACTURER Murata Electronics -> (none); KiLib_Generator SMD_2terminal_chip_molded -> (none); LCSC MANUFACTURER HRE -> (none); LCSC PN C6119795 -> (none); LCSC_PN (none) -> C368809; MOUSER_PN (none) -> 810-C1005X5R1A475KBC; PN CGA0402X5R475M250GT -> C1005X5R1A475K050BC
- C14, C15: value 12pF -> 27pF; DIGIKEY_PN (none) -> 490-5869-1-ND; LCSC_PN (none) -> C1557; MOUSER_PN (none) -> 81-GRM1555C1H270JA1D; PN (none) -> GRM1555C1H270JA01D; Tolerance (none) -> ±5%
- D1: DIGIKEY PN 732-4971-1-ND -> (none); DIGIKEY_PN (none) -> 160-LTST-C190GKTCT-ND; DIGKEY MANUFACTURER Würth Elektronik -> (none); KiLib_Generator SMD_2terminal_chip_molded -> (none); LCSC MANUFACTURER EVERLIGHT -> (none); LCSC PN C2986048 -> (none); LCSC_PN (none) -> C125094; MOUSER_PN (none) -> 859-LTST-C190GKT; PN 19-21/GHC-YR1S2/4T -> LTST-C190GKT
- FB100: value MLB1005F-221T -> MPZ1005S221HT000; DIGIKEY PN 445-6404-1-ND -> (none); DIGIKEY_PN (none) -> 445-MPZ1005S221HT000CT-ND; DIGKEY MANUFACTURER TDK -> (none); KiLib_Generator SMD_2terminal_chip_molded -> (none); LCSC MANUFACTURER MetalLions -> (none); MOUSER_PN (none) -> 810-MPZ1005S221HT000
- J1: value 1.0-3PWT -> SM03B-SRSS-TB; DIGIKEY PN 455-SM03B-SRSS-TBCT-ND -> (none); DIGIKEY_PN (none) -> 455-SM03B-SRSS-TBCT-ND; DIGKEY MANUFACTURER JST Sales America Inc. -> (none); KiLib_Generator connector/SMD_single_row_plus_mounting_pad -> (none); LCSC MANUFACTURER FG -> (none); LCSC PN C2763613 -> (none); LCSC_PN (none) -> C7430445
- L3: DIGIKEY PN 535-AOTA-B201610S3R3-101-TCT-ND -> (none); DIGIKEY_PN (none) -> 535-AOTA-B201610S3R3-101-TCT-ND; DIGKEY MANUFACTURER Abracon LLC -> (none); LCSC MANUFACTURER ABRACON -> (none); MOUSER_PN (none) -> 815-AB201610S3R3101T
- R1, R2: DIGIKEY PN 311-100LRCT-ND -> (none); DIGIKEY_PN (none) -> 311-100LRCT-ND; DIGKEY MANUFACTURER YAGEO -> (none); KiLib_Generator SMD_2terminal_chip_molded -> (none); LCSC MANUFACTURER CHANGLONG -> (none); LCSC PN C46635166 -> (none); LCSC_PN (none) -> C106232; MOUSER_PN (none) -> 603-RC0402FR-07100RL; PN CL0402FN100RP -> RC0402FR-07100RL
- R13: DIGIKEY PN 13-RC0402FR-131K1LCT-ND -> (none); DIGIKEY_PN (none) -> 311-620LRCT-ND; DIGKEY MANUFACTURER YAGEO -> (none); KiLib_Generator SMD_2terminal_chip_molded -> (none); LCSC MANUFACTURER FOJAN -> (none); LCSC PN C2909306 -> (none); LCSC_PN (none) -> C413077; MOUSER_PN (none) -> 603-RC0402FR-07620RL; PN FRC0402F1101TS -> RC0402FR-07620RL
- R3, R4, R5: DIGIKEY PN YAG3086CT-ND -> (none); DIGIKEY_PN (none) -> YAG3086CT-ND; DIGKEY MANUFACTURER YAGEO -> (none); KiLib_Generator SMD_2terminal_chip_molded -> (none); LCSC MANUFACTURER FOJAN -> (none); LCSC PN C2909343 -> (none); LCSC_PN (none) -> C2909343; MOUSER_PN (none) -> 603-RC0402FR-0727RL; PN FRC0402F27R0TS -> RC0402FR-0727RL
- R46: DIGIKEY PN 13-RC0402FR-131K1LCT-ND -> (none); DIGIKEY_PN (none) -> 311-1.10KLRCT-ND; DIGKEY MANUFACTURER YAGEO -> (none); KiLib_Generator SMD_2terminal_chip_molded -> (none); LCSC MANUFACTURER FOJAN -> (none); LCSC PN C2909306 -> (none); LCSC_PN (none) -> C2909306; MOUSER_PN (none) -> 603-RC0402FR-071K1L; PN FRC0402F1101TS -> RC0402FR-071K1L
- U1: DIGIKEY PN 2648-SC1510-A4CT-ND -> (none); DIGIKEY_PN (none) -> 2648-SC1510-A4CT-ND; DIGKEY MANUFACTURER Raspberry Pi -> (none); KiLib_Generator package/no_lead -> (none); LCSC MANUFACTURER Raspberry PI -> (none); MOUSER_PN (none) -> 358-SC1510; PN ${VALUE} -> SC1510-A4
- Y1: DIGIKEY PN 535-10261-1-ND -> (none); DIGIKEY_PN (none) -> 535-10261-1-ND; DIGKEY MANUFACTURER Abracon LLC -> (none); LCSC_PN (none) -> C596904; MOUSER_PN (none) -> 815-ABM8G-12-18D2Y
