File: phyduino_pico2.kicad_sch (KiCad schematic)
At the start: 16 parts, among them J2 PPPC081LFBN-RC, J3 PPPC101LFBN-RC, J4 PPPC061LFBN-RC, J5 PPPC081LFBN-RC, J6 GT-USB-7047A, J7 HC-FPC-0.5-22P-CSH20, J8 54-00127, J9 SM04B-SRSS-TB, U9 TPUSBLC6-2P6

Commit message: Development update : Schematic review changes (findings #6-#26).
- Pin map reworked onto 5 V-tolerant GPIOs; I2C1 shared by EEPROM,
  expander and J7 on GPIO38/39; UART1 shared by D0/D1 and ESP32 flashing.
- Power: U10 enable on GPIO33 (EN_5V) with VIN_MONITOR on GPIO43;
  VIN works like an Uno's (J2.8 on +V_EXTERNAL, U12 removed); C22 moved
  to +5.0V; C134 added on +V_EXTERNAL; C27 10 uF, C140 3.3 nF; notes
  corrected.
- A0-A5 protected with 1 kOhm arrays and 1 nF; R53 pull-down on WIFI_ENA;
  32 kHz labels removed; Y1 ABM8G with 12 pF load caps; I2C address
  notes corrected; Variants set on all parts.

Co-Authored-By: Claude Opus 5.5 <noreply@anthropic.com>
Parts:
- C27: value 22µF -> 10µF; DIGIKEY PN 1276-CL21A226MAYNNNECT-ND -> (none); DIGKEY MANUFACTURER Samsung Electro-Mechanics -> (none); KiLib_Generator SMD_2terminal_chip_molded -> (none); LCSC MANUFACTURER Chinocera -> (none); LCSC PN C22367832 -> (none); PN HGC0805R5226M350NSLJ -> (none)
- J2, J3, J4: KiLib_Generator (none) -> connector/pin_header_socket
- J5: KiLib_Generator (none) -> connector/pin_header_socket; LCSC PN (none) -> C5224027
- J9: KiLib_Generator (none) -> connector/SMD_single_row_plus_mounting_pad; Variant (none) -> ADV_SMT
Connections:
- net +V_{IN} is gone; now on net +V_{EXTERNAL}: J2.8 (Pin_8)
- net Microcontroller/HS_I2C1_SCL renamed Microcontroller/I2C1_SCL
- net Microcontroller/HS_I2C1_SDA renamed Microcontroller/I2C1_SDA
Other:
- sheet Microcontroller ports: added EN_5V, I2C1_SCL, I2C1_SDA, VIN_MONITOR; removed HS_I2C1_SCL, HS_I2C1_SDA, SHIELD_AUXOFF, SHIELD_~{FLT}
- sheet Power ports: added EN_5V, VIN_MONITOR; removed +SHIELD_VIN, SHIELD_AUXOFF, SHIELD_~{FLT}
