File: phyduino_pico2.kicad_sch (KiCad schematic)
At the start: 18 parts, among them J2 PPPC081LFBN-RC, J3 PPPC101LFBN-RC, J4 PPPC061LFBN-RC, J5 PPPC081LFBN-RC, J6 GT-USB-7047A, J7 HC-FPC-0.5-22P-CSH20, J8 54-00127, J9 SM04B-SRSS-TB, U9 TPUSBLC6-2P6

Commit message: Updated part numbers and distributor part nummbers after BoM review.
Parts:
- C27: DIGIKEY_PN (none) -> 587-4893-1-ND; LCSC_PN (none) -> C440198; MOUSER_PN (none) -> 603-CC0805KKX59BB106; PN (none) -> GMK212BBJ106KG-T; Tolerance (none) -> ±10%
- C39: DIGIKEY PN 490-GRM155C61E475ME15DCT-ND -> (none); DIGIKEY_PN (none) -> 1276-1067-1-ND; DIGKEY MANUFACTURER Murata Electronics -> (none); KiLib_Generator SMD_2terminal_chip_molded -> (none); LCSC MANUFACTURER HRE -> (none); LCSC PN C6119795 -> (none); LCSC_PN (none) -> C29266; MOUSER_PN (none) -> 187-CL05A105KO5NNNC; PN CGA0402X5R475M250GT -> CL05A105KO5NNNC
- C9: footprint Capacitor_SMD:C_1206_3216Metric_Pad1.33x1.80mm_HandSolder -> Capacitor_SMD:C_1210_3225Metric; DIGIKEY PN 399-C1206C104K5RACTUCT-ND -> (none); DIGIKEY_PN (none) -> 399-C1210C104KCRACTUCT-ND; DIGKEY MANUFACTURER KEMET -> (none); KiLib_Generator SMD_2terminal_chip_molded -> (none); LCSC MANUFACTURER HRE -> (none); LCSC PN C22374889 -> (none); LCSC_PN (none) -> C141218; MOUSER_PN (none) -> 80-C1210C104KCRACTU; PN CGA1206X7R104K501NT -> C1210C104KCRACTU; Tolerance (none) -> ±10%; VOLTAGE (none) -> 500V
- H2: KiLib_Generator mounting_hardware/mounting_hole -> (none)
- J2, J5: DIGIKEY_PN (none) -> S7041-ND; KiLib_Generator connector/pin_header_socket -> (none)
- J3: DIGIKEY_PN (none) -> S7043-ND; KiLib_Generator connector/pin_header_socket -> (none)
- J4: DIGIKEY_PN (none) -> S7039-ND; KiLib_Generator connector/pin_header_socket -> (none)
- J6: value GT-USB-7047A -> USB4110-GF-A; DIGIKEY PN 2073-USB4110-GF-A-1-ND -> (none); DIGIKEY_PN (none) -> 2073-USB4110-GF-A-1-ND; DIGKEY MANUFACTURER GCT -> (none); LCSC MANUFACTURER G-Switch -> (none); LCSC PN C963216 -> (none); LCSC_PN (none) -> C5143397; MOUSER_PN (none) -> 640-USB4110-GF-A
- J7: value HC-FPC-0.5-22P-CSH20 -> F32Q-1A7H1-11022; DIGIKEY PN 609-F32Q-1A7H1-11022CT-ND -> (none); DIGIKEY_PN (none) -> 609-F32Q-1A7H1-11022CT-ND; DIGKEY MANUFACTURER Amphenol ICC (FCI) -> (none); KiLib_Generator connector/Amphenol -> (none); LCSC MANUFACTURER Hong Cheng -> (none); MOUSER_PN (none) -> 649-F32Q-1A7H1-11022
- J8: DIGIKEY_PN (none) -> 839-54-00127-ND; PN (none) -> ${VALUE}
- J9: DIGIKEY_PN (none) -> 455-SM04B-SRSS-TBCT-ND; KiLib_Generator connector/SMD_single_row_plus_mounting_pad -> (none); LCSC_PN (none) -> C160404; MOUSER_PN (none) -> 306-SM04BSRSSTBLFSN; PN (none) -> ${VALUE}
- R164: DIGIKEY PN 311-10.0KLRCT-ND -> (none); DIGIKEY_PN (none) -> 311-10.0KLRCT-ND; DIGKEY MANUFACTURER YAGEO -> (none); KiLib_Generator SMD_2terminal_chip_molded -> (none); LCSC MANUFACTURER FOJAN -> (none); LCSC PN C2906861 -> (none); LCSC_PN (none) -> C60490; MOUSER_PN (none) -> 603-RC0402FR-0710KL; PN FRC0402F1002TS -> RC0402FR-0710KL
- R47, R48: DIGIKEY PN 13-RC0402FR-7W5K1LCT-ND -> (none); DIGIKEY_PN (none) -> 311-5.10KLRCT-ND; DIGKEY MANUFACTURER YAGEO -> (none); KiLib_Generator SMD_2terminal_chip_molded -> (none); LCSC MANUFACTURER CHANGLONG -> (none); LCSC PN CHANGLONG -> (none); LCSC_PN (none) -> C105872; MOUSER_PN (none) -> 603-RC0402FR-075K1L; PN CHANGLONG -> RC0402FR-075K1L
- R6: DIGIKEY PN 13-RC0805FR-13220KLCT-ND -> (none); DIGIKEY_PN (none) -> 311-220KCRCT-ND; DIGKEY MANUFACTURER YAGEO -> (none); KiLib_Generator SMD_2terminal_chip_molded -> (none); LCSC MANUFACTURER FOJAN -> (none); LCSC PN C2907242 -> (none); LCSC_PN (none) -> C137568; MOUSER_PN (none) -> 603-RC0805FR-07220KL; PN FRC0805F2203TS -> RC0805FR-07220KL
- R65: DIGIKEY_PN (none) -> 311-5.10KLRCT-ND; KiLib_Generator SMD_2terminal_chip_molded -> (none); LCSC_PN (none) -> C105872; MOUSER_PN (none) -> 603-RC0402FR-075K1L; PN (none) -> RC0402FR-075K1L
- U9: value TPUSBLC6-2P6 -> USBLC6-2P6; DIGIKEY PN 497-5026-1-ND -> (none); DIGIKEY_PN (none) -> 497-5026-1-ND; DIGKEY MANUFACTURER STMicroelectronics -> (none); LCSC MANUFACTURER TECH PUBLIC -> (none); LCSC PN C2682291 -> (none); LCSC_PN (none) -> C2827693; MOUSER_PN (none) -> 511-USBLC6-2P6
