File: phyduino_pico2_wifi.kicad_sch (KiCad schematic)
At the start: 10 parts, among them U11 ESP32-C6-MINI-1-H4

Commit message: Development update : Schematic review changes (findings #6-#26).
- Pin map reworked onto 5 V-tolerant GPIOs; I2C1 shared by EEPROM,
  expander and J7 on GPIO38/39; UART1 shared by D0/D1 and ESP32 flashing.
- Power: U10 enable on GPIO33 (EN_5V) with VIN_MONITOR on GPIO43;
  VIN works like an Uno's (J2.8 on +V_EXTERNAL, U12 removed); C22 moved
  to +5.0V; C134 added on +V_EXTERNAL; C27 10 uF, C140 3.3 nF; notes
  corrected.
- A0-A5 protected with 1 kOhm arrays and 1 nF; R53 pull-down on WIFI_ENA;
  32 kHz labels removed; Y1 ABM8G with 12 pF load caps; I2C address
  notes corrected; Variants set on all parts.

Co-Authored-By: Claude Opus 5.5 <noreply@anthropic.com>
Parts:
- added R53: 10kΩ, Resistor_SMD:R_0402_1005Metric, symbol phyduino_pico:R_Small
- added TP11: TestPoint_Small, Component - Test point SMT [UL]:TestPoint_SameSky_CPG-47-TH-B, symbol Connector [KL]:TestPoint_Small
- renumbered TP14 to TP1, TP9 to TP2, TP8 to TP3
Connections:
- net GND: now also R53.2
- net WIFI_BOOT1: now also TP11.1
- net WIFI_ENA: now also R53.1
- net XTAL_32K_N: no longer names the net of U11.13 (IO1)
- net XTAL_32K_P: no longer names the net of U11.12 (IO0)
- no-connect marks 12 -> 14
