File: phyduino_pico_peripherals.kicad_sch (KiCad schematic)
At the start: 25 parts, among them U14 FXL6408UMX, U5 ADS7038QRTERQ1, U7 24AA64FT-I/MNY

Commit message: Updated part numbers and distributor part nummbers after BoM review.
Parts:
- C10, C11, C12: DIGIKEY_PN (none) -> 490-10675-1-ND; KiLib_Generator SMD_2terminal_chip_molded -> (none); LCSC_PN (none) -> C342759; MOUSER_PN (none) -> 81-GCM21BR71H105KA3L; PN (none) -> GCM21BR71H105KA03L; Tolerance (none) -> ±10%
- C21, C29: DIGIKEY PN 490-14514-1-ND -> (none); DIGIKEY_PN (none) -> 490-14514-1-ND; DIGKEY MANUFACTURER Murata Electronics -> (none); KiLib_Generator SMD_2terminal_chip_molded -> (none); LCSC MANUFACTURER CCTC -> (none); LCSC PN C5142567 -> (none); LCSC_PN (none) -> C85858; MOUSER_PN (none) -> 81-GCM155R71H104KE2J; PN TCC0402X7R104M500AT -> GCM155R71H104KE02J; Tolerance (none) -> ±10%
- C30, C31, C32, C33, C35, C38: DIGIKEY_PN (none) -> 490-3244-1-ND; KiLib_Generator SMD_2terminal_chip_molded -> (none); LCSC_PN (none) -> C76947; MOUSER_PN (none) -> 81-GRM1555C1H102JA1D; PN (none) -> GRM1555C1H102JA01D; Tolerance (none) -> ±5%
- FB1: value (none) -> 1kΩ@100MHz; DIGIKEY_PN (none) -> 240-2397-1-ND; KiLib_Generator SMD_2terminal_chip_molded -> (none); LCSC_PN (none) -> C85835; MOUSER_PN (none) -> 875-HZ0805D102R-10; PN ${VALUE} -> HZ0805D102R-10
- R42, R43, R61, R62: DIGIKEY_PN (none) -> 311-5.10KLRCT-ND; KiLib_Generator SMD_2terminal_chip_molded -> (none); LCSC_PN (none) -> C105872; MOUSER_PN (none) -> 603-RC0402FR-075K1L; PN (none) -> RC0402FR-075K1L
- R63, R64: DIGIKEY_PN (none) -> 311-10.0KLRCT-ND; KiLib_Generator SMD_2terminal_chip_molded -> (none); LCSC_PN (none) -> C60490; MOUSER_PN (none) -> 603-RC0402FR-0710KL; PN (none) -> RC0402FR-0710KL
- RN1, RN2: DIGIKEY_PN (none) -> CAT10-102J4LFCT-ND; MOUSER_PN (none) -> 652-CAT10-102J4LF
- U14: DIGIKEY_PN (none) -> FXL6408UMXCT-ND; LCSC_PN (none) -> C457770; MFR ON Semiconductor -> (none); MOUSER_PN (none) -> 512-FXL6408UMX; PN FXL6408UMX -> ${VALUE}
- U5: value ADS7038QRTERQ1 -> ADS7038IRTER; DIGIKEY PN 296-ADS7038QRTERQ1CT-ND -> (none); DIGIKEY_PN (none) -> 296-ADS7038IRTERCT-ND; DIGKEY MANUFACTURER Texas Instruments -> (none); LCSC MANUFACTURER Texas Instruments -> (none); LCSC PN C2876384 -> (none); LCSC_PN (none) -> C2871580; MOUSER_PN (none) -> 595-ADS7038IRTER
- U7: value 24AA64FT-I/MNY -> AT24C64D-MAHM-T; DIGIKEY PN 24AA64FT-I/MNYCT-ND -> (none); DIGIKEY_PN (none) -> AT24C64D-MAHM-TCT-ND; DIGKEY MANUFACTURER Microchip Technology -> (none); LCSC_PN (none) -> C2061553
