File: phyduino_pico_memory.kicad_sch (KiCad schematic)
At the start: 18 parts, among them SW1 1977067-1, U15 TPS3424C11EF2ADRLR, U2 AT25QF128A-SHB-T, U3 IS66WVR8M8FBLL-104NLI

Commit message: Updated part numbers and distributor part nummbers after BoM review.
Parts:
- C1, C20, C57, C6: DIGIKEY PN 490-14514-1-ND -> (none); DIGIKEY_PN (none) -> 490-14514-1-ND; DIGKEY MANUFACTURER Murata Electronics -> (none); KiLib_Generator SMD_2terminal_chip_molded -> (none); LCSC MANUFACTURER CCTC -> (none); LCSC PN C5142567 -> (none); LCSC_PN (none) -> C85858; MOUSER_PN (none) -> 81-GCM155R71H104KE2J; PN TCC0402X7R104M500AT -> GCM155R71H104KE02J; Tolerance (none) -> ±10%
- C58: DIGIKEY PN 490-14514-1-ND -> (none); DIGIKEY_PN (none) -> 490-GRM1555C1H472JE01DCT-ND; DIGKEY MANUFACTURER Murata Electronics -> (none); KiLib_Generator SMD_2terminal_chip_molded -> (none); LCSC MANUFACTURER CCTC -> (none); LCSC PN C5142567 -> (none); LCSC_PN (none) -> C1518204; MOUSER_PN (none) -> 81-GRM1555C1H472JE1D; PN TCC0402X7R104M500AT -> GRM1555C1H472JE01D; Tolerance (none) -> ±5%
- C59: DIGIKEY_PN (none) -> 490-3244-1-ND; LCSC MANUFACTURER CCTC -> (none); LCSC PN C5142567 -> (none); LCSC_PN (none) -> C76947; MOUSER_PN (none) -> 81-GRM1555C1H102JA1D; PN (none) -> GRM1555C1H102JA01D; Tolerance (none) -> ±5%
- R20, R21, R22: DIGIKEY PN 311-10.0KLRCT-ND -> (none); DIGIKEY_PN (none) -> 311-10.0KLRCT-ND; DIGKEY MANUFACTURER YAGEO -> (none); KiLib_Generator SMD_2terminal_chip_molded -> (none); LCSC MANUFACTURER FOJAN -> (none); LCSC PN C2906861 -> (none); LCSC_PN (none) -> C60490; MOUSER_PN (none) -> 603-RC0402FR-0710KL; PN FRC0402F1002TS -> RC0402FR-0710KL
- R49, R51, R52: DIGIKEY PN 13-RC0402FR-7W5K1LCT-ND -> (none); DIGIKEY_PN (none) -> 311-10.0KLRCT-ND; DIGKEY MANUFACTURER YAGEO -> (none); KiLib_Generator SMD_2terminal_chip_molded -> (none); LCSC MANUFACTURER CHANGLONG -> (none); LCSC PN CHANGLONG -> (none); LCSC_PN (none) -> C60490; MOUSER_PN (none) -> 603-RC0402FR-0710KL; PN CHANGLONG -> RC0402FR-0710KL
- SW1: DIGIKEY PN 450-1977067-1DKR-ND -> (none); DIGIKEY_PN (none) -> 450-1977067-1CT-ND; DIGKEY MANUFACTURER TE Connectivity ALCOSWITCH Switches -> (none); LCSC MANUFACTURER TE Connectivity -> (none)
- U15: DIGIKEY_PN (none) -> 296-TPS3424C11EF2ADRLRCT-ND; MOUSER_PN (none) -> 595-S3424C11EF2ADRLR; PN (none) -> ${VALUE}
- U2: DIGIKEY_PN (none) -> 1695-AT25QF128A-SHB-TCT-ND; KiLib_Generator package/gullwing -> (none); LCSC_PN (none) -> C7452501; MOUSER_PN (none) -> 988-AT25QF128A-SHB-T; PN (none) -> ${VALUE}
- U3: value IS66WVR8M8FBLL-104NLI -> IS66WVS8M8FBLL-104NLI; DIGIKEY_PN (none) -> 706-IS66WVS8M8FBLL-104NLI-ND; KiLib_Generator package/gullwing -> (none); MOUSER_PN (none) -> 870-WVS8M8FBLL104NLI; PN (none) -> ${VALUE}

Commit message: DRC check changes and fabracation output.
Other:
- note added: "Long button press is ~2sec Short button press is 50ms (default DNP)"
- moved on the sheet: C57, SW1
